File: Shield/Htr_Fan.sch (KiCad schematic (older format))
At the start: 30 parts, among them J27 TP

Commit message: All schematic connections to the stepper drivers, heaters, and thermistors complete.
Parts:
- removed D8: LED, symbol LED
- removed R24: 470R, symbol R
- removed R25: 220R, symbol R
- removed R68: 4k7, symbol R
- removed R79: 100k, symbol R
- removed TR5: BSH105, symbol BSH105
- removed TR6: IPD036N04L, symbol IPD036N04L
Connections:
- net labels added: E1-, E1_PWM, E1_THERMISTOR, E2-, E2_PWM, E2_THERMISTOR
- net labels removed: BED-, BED_PWM, BED_THERMISTOR, E0-, E0_PWM, E0_THERMISTOR, FAN0-, FAN0_PWM
- wire segments 87 -> 67
Other:
- note added: "E1 MOSFET CONTROL"
- note added: "E2 MOSFET CONTROL"
- note removed: "BED MOSFET CONTROL"
- note removed: "E0 MOSFET CONTROL"
- note removed: "FAN MOSFET CONTROL"
Changed lines of the file:
@@
-EESchema Schematic File Version 2  date 19/07/2014 15:49:20
+EESchema Schematic File Version 2  date Thu 06 Nov 2014 10:06:04 GMT
 LIBS:power
 LIBS:device
@@
 LIBS:valves
 LIBS:FE
-LIBS:Duet0.7-cache
+LIBS:Shield-cache
 EELAYER 25  0
 EELAYER END
@@
 Sheet 6 7
 Title "Duet"
-Date "19 jul 2014"
+Date "5 nov 2014"
 Rev "0.7"
 Comp "Think3DPrint3D, RepRapPro"
@@
 	2600 2850 2250 2850
 Wire Wire Line
-	10950 2900 10950 2850
-Wire Wire Line
-	10950 2850 10550 2850
-Wire Wire Line
 	6750 2900 6750 2850
 Wire Wire Line
 	6750 2850 6350 2850
-Wire Wire Line
-	9950 2100 9950 1800
-Connection ~ 9950 3500
-Wire Wire Line
-	10100 3500 9850 3500
 Wire Wire Line
 	5750 2600 5750 3500
@@
 Wire Wire Line
 	7400 1800 7400 1850
-Wire Wire Line
-	11300 2400 11300 2500
 Connection ~ 7400 2950
 Wire Wire Line
@@
 Wire Wire Line
 	2750 5600 3550 5600
-Wire Wire Line
-	11600 3100 11600 2200
-Wire Wire Line
-	10550 3850 10550 4300
-Wire Wire Line
-	10550 3150 10550 2600
-Connection ~ 10550 2850
-Wire Wire Line
-	11600 2200 12150 2200
-Wire Wire Line
-	10550 1800 10550 2100
 Wire Wire Line
 	6350 1800 6350 2100
@@
 Wire Wire Line
 	2750 7100 2750 6900
-Wire Notes Line
-	9250 1250 12750 1250
-Wire Notes Line
-	9250 1250 9250 4750
-Wire Notes Line
-	9250 4750 12750 4750
-Wire Notes Line
-	12750 4750 12750 1250
 Wire Notes Line
 	8550 4750 8550 1250
@@
 Connection ~ 3300 2950
 Wire Wire Line
-	11600 3800 11600 4450
-Wire Wire Line
 	7100 2400 7100 2500
-Wire Wire Line
-	11300 1900 11300 1850
-Wire Wire Line
-	11300 1850 11600 1850
-Wire Wire Line
-	11300 2900 11300 3000
-Wire Wire Line
-	11300 3000 11600 3000
-Connection ~ 11600 3000
-Wire Wire Line
-	11600 1850 11600 1800
 Wire Wire Line
 	3300 1800 3300 1850
@@
 	5750 1800 5750 2100
 Wire Wire Line
-	10550 4300 11600 4300
-Connection ~ 11600 4300
-Wire Wire Line
-	9950 2600 9950 3500
-Wire Wire Line
 	3300 4300 1650 4300
 Connection ~ 2250 4300
@@
 Wire Wire Line
 	6750 3450 6950 3450
-Wire Wire Line
-	10950 3400 10950 3450
-Wire Wire Line
-	10950 3450 11150 3450
 Wire Wire Line
 	2600 3400 2600 3450
@@
 $EndComp
 $Comp
-L R R25
-U 1 1 53B06825
-P 10950 3150
-F 0 "R25" V 11030 3150 50  0000 C CNN
-F 1 "220R" V 10950 3150 50  0000 C CNN
-	1    10950 3150
-	1    0    0    -1
-$EndComp
-$Comp
 L R R23
 U 1 1 53B0680C
@@
 	1    1650 4300
 	1    0    0    -1
-$EndComp
-$Comp
-L R R79
-U 1 1 522617BB
-P 9950 2350
-F 0 "R79" V 10030 2350 50  0000 C CNN
-F 1 "100k" V 9950 2350 50  0000 C CNN
-	1    9950 2350
-	-1   0    0    1
 $EndComp
 $Comp
@@
 Text GLabel 3150 7200 3    60   Input ~ 0
 VSSA
-$Comp
-L LED D8
-U 1 1 50905423
-P 11300 2700
-F 0 "D8" H 11300 2800 50  0000 C CNN
-F 1 "LED" H 11300 2600 50  0000 C CNN
-	1    11300 2700
-	0    1    1    0
-$EndComp
-Text GLabel 9950 1800 1    60   Input ~ 0
-+3.3V
-$Comp
-L IPD036N04L TR6
-U 1 1 50905422
-P 11450 3450
-F 0 "TR6" H 11900 3550 70  0000 C CNN
-F 1 "IPD036N04L" H 11950 3350 60  0000 C CNN
-	1    11450 3450
-	1    0    0    -1
-$EndComp
-$Comp
-L BSH105 TR5
-U 1 1 50905421
-P 10400 3500
-F 0 "TR5" H 10303 3750 70  0000 C CNN
-F 1 "BSH105" H 10253 3203 60  0000 C CNN
-	1    10400 3500
-	1    0    0    -1
-$EndComp
-Text GLabel 12150 2200 2    60   Input ~ 0
-FAN0-
-$Comp
-L GND #PWR056
-U 1 1 5090541F
-P 11600 4450
-F 0 "#PWR056" H 11600 4450 30  0001 C CNN
-F 1 "GND" H 11600 4380 30  0001 C CNN
-	1    11600 4450
-	1    0    0    -1
-$EndComp
-$Comp
-L R R24
-U 1 1 5090541E
-P 10550 2350
-F 0 "R24" V 10630 2350 50  0000 C CNN
-F 1 "470R" V 10550 2350 50  0000 C CNN
-	1    10550 2350
-	1    0    0    -1
-$EndComp
-Text GLabel 9850 3500 0    60   Input ~ 0
-FAN0_PWM
-Text GLabel 11600 1800 1    60   Input ~ 0
-V_IN
-Text GLabel 10550 1800 1    60   Input ~ 0
-+5V
 Text GLabel 6350 1800 1    60   Input ~ 0
 +5V
@@
 V_IN
 Text GLabel 5600 3500 0    60   Input ~ 0
-E0_PWM
+E2_PWM
 $Comp
 L R R22
@@
 $EndComp
 Text GLabel 7450 2200 2    60   Input ~ 0
-E0-
+E2-
 $Comp
 L BSH105 TR3
@@
 $EndComp
 $Comp
-L R R68
-U 1 1 50905410
-P 11300 2150
-F 0 "R68" V 11380 2150 50  0000 C CNN
-F 1 "4k7" V 11300 2150 50  0000 C CNN
-	1    11300 2150
-	-1   0    0    1
-$EndComp
-$Comp
 L R R65
 U 1 1 5090334F
@@
 $EndComp
 Text GLabel 4400 6400 2    60   Input ~ 0
-BED_THERMISTOR
+E2_THERMISTOR
 Text GLabel 1950 6400 0    60   Input ~ 0
-E0_THERMISTOR
+E1_THERMISTOR
 $Comp
 L IPD036N04L TR2
@@
 Text Notes 1150 5250 0    60   ~ 0
 THERMISTOR INPUTS
-Text Notes 9300 1400 0    60   ~ 0
-FAN MOSFET CONTROL
 Text Notes 5100 1400 0    60   ~ 0
-E0 MOSFET CONTROL
+E2 MOSFET CONTROL
 Text Notes 1000 1400 0    60   ~ 0
-BED MOSFET CONTROL
+E1 MOSFET CONTROL
 Text GLabel 3300 2200 2    60   Input ~ 0
-BED-
+E1-
 $Comp
 L GND #PWR058
@@
 $EndComp
 Text GLabel 1500 3500 0    60   Input ~ 0
-BED_PWM
+E1_PWM
 Text GLabel 3300 1800 1    60   Input ~ 0
 V_IN

Commit message: Inputs and outputs tidied to keep DRC a bit happier...
Changed lines of the file:
@@
-EESchema Schematic File Version 2  date Thu 06 Nov 2014 16:31:39 GMT
+EESchema Schematic File Version 2  date Fri 07 Nov 2014 11:38:16 GMT
 LIBS:power
 LIBS:device
@@
 $Descr A3 16535 11700
 encoding utf-8
-Sheet 6 4
+Sheet 4 4
 Title "Duet"
-Date "6 nov 2014"
+Date "7 nov 2014"
 Rev "0.7"
 Comp "Think3DPrint3D, RepRapPro"
@@
 $EndComp
 $Comp
-L GND #PWR057
+L GND #PWR048
 U 1 1 50905416
 P 7400 4450
-F 0 "#PWR057" H 7400 4450 30  0001 C CNN
+F 0 "#PWR048" H 7400 4450 30  0001 C CNN
 F 1 "GND" H 7400 4380 30  0001 C CNN
 	1    7400 4450
 	1    0    0    -1
 $EndComp
-Text GLabel 7450 2200 2    60   Input ~ 0
+Text GLabel 7450 2200 2    60   Output ~ 0
 E2-
 $Comp
@@
 Text Notes 1000 1400 0    60   ~ 0
 E1 MOSFET CONTROL
-Text GLabel 3300 2200 2    60   Input ~ 0
+Text GLabel 3300 2200 2    60   Output ~ 0
 E1-
 $Comp
-L GND #PWR058
+L GND #PWR049
 U 1 1 5064BB75
 P 3300 4450
-F 0 "#PWR058" H 3300 4450 30  0001 C CNN
+F 0 "#PWR049" H 3300 4450 30  0001 C CNN
 F 1 "GND" H 3300 4380 30  0001 C CNN
 	1    3300 4450
