File: Shield/Stepper_Drv.sch (KiCad schematic (older format))
At the start: 110 parts, among them J16 VREF, J17 VREF, J18 VREF, J3 VREF, U5 A4982SLPTR, U6 A4982SLPTR, U7 A4982SLPTR, U8 A4982SLPTR, U9 MCP44X1

Commit message: All schematic connections to the stepper drivers, heaters, and thermistors complete.
Connections:
- net labels added: E1_DIR, E1_EN, E1_MOT_1A, E1_MOT_1B, E1_MOT_2A, E1_MOT_2B, E1_REF, E1_STEP, E1_STOP, E1_STOP_CONN, E2_DIR, E2_EN, E2_MOT_1A, E2_MOT_1B, E2_MOT_2A, E2_MOT_2B, E2_REF, E2_STEP, E2_STOP, E2_STOP_CONN, E3_DIR, E3_EN, E3_MOT_1A, E3_MOT_1B, E3_MOT_2A, E3_MOT_2B, E3_REF, E3_STEP, E3_STOP, E3_STOP_CONN, E4_DIR, E4_EN, E4_MOT_1A, E4_MOT_1B, E4_MOT_2A, E4_MOT_2B, E4_REF, E4_STEP, E4_STOP, E4_STOP_CONN
- net labels removed: E0_DIR, E0_EN, E0_MOT_1A, E0_MOT_1B, E0_MOT_2A, E0_MOT_2B, E0_REF, E0_STEP, E0_STOP, E0_STOP_CONN, X_DIR, X_EN, X_MOT_1A, X_MOT_1B, X_MOT_2A, X_MOT_2B, X_REF, X_STEP, X_STOP, X_STOP_CONN, Y_DIR, Y_EN, Y_MOT_1A, Y_MOT_1B, Y_MOT_2A, Y_MOT_2B, Y_REF, Y_STEP, Y_STOP, Y_STOP_CONN, Z_DIR, Z_EN, Z_MOT_1A, Z_MOT_1B, Z_MOT_2A, Z_MOT_2B, Z_REF, Z_STEP, Z_STOP, Z_STOP_CONN
Other:
- note added: "E1 Stepper Driver"
- note added: "E2 Stepper Driver"
- note added: "E3 Stepper Driver"
- note added: "E4 Stepper Driver"
- note removed: "Extruder Stepper Driver"
- note removed: "X-Axis Stepper Driver"
- note removed: "Y-Axis Stepper Driver"
- note removed: "Z-Axis Stepper Driver"
Changed lines of the file:
@@
-EESchema Schematic File Version 2  date 13/07/2014 12:00:17
+EESchema Schematic File Version 2  date Thu 06 Nov 2014 10:06:04 GMT
 LIBS:power
 LIBS:device
@@
 LIBS:valves
 LIBS:FE
-LIBS:Duet0.7-cache
+LIBS:Shield-cache
 EELAYER 25  0
 EELAYER END
@@
 Sheet 2 7
 Title "Duet"
-Date "13 jul 2014"
+Date "5 nov 2014"
 Rev "0.7"
 Comp "Think3DPrint3D, RepRapPro"
@@
 +3.3V
 Text GLabel 14050 9150 0    39   Output ~ 0
-E0_STOP
+E4_STOP
 Text GLabel 12150 9150 0    39   Output ~ 0
-Z_STOP
+E3_STOP
 Text GLabel 14050 6550 0    39   Output ~ 0
-X_STOP
+E1_STOP
 Text GLabel 12150 6550 0    39   Output ~ 0
-Y_STOP
+E2_STOP
 Text GLabel 13000 7800 1    39   Input ~ 0
 +3.3V
@@
 $EndComp
 Text GLabel 13200 9150 2    39   Output ~ 0
-Z_STOP_CONN
+E3_STOP_CONN
 $Comp
 L R_SMALL R58
@@
 $EndComp
 Text GLabel 15050 9150 2    39   Output ~ 0
-E0_STOP_CONN
+E4_STOP_CONN
 Text GLabel 13200 6550 2    39   Output ~ 0
-Y_STOP_CONN
+E2_STOP_CONN
 $Comp
 L R_SMALL R57
@@
 $EndComp
 Text GLabel 15100 6550 2    39   Output ~ 0
-X_STOP_CONN
+E1_STOP_CONN
 $Comp
 L R_SMALL R51
@@
 Digital Current Limit Control
 Text Notes 5700 6200 2    60   ~ 0
-Z-Axis Stepper Driver
+E3 Stepper Driver
 Text Notes 11000 6200 2    60   ~ 0
-Extruder Stepper Driver
+E4 Stepper Driver
 Text Notes 11000 1000 2    60   ~ 0
-Y-Axis Stepper Driver
+E2 Stepper Driver
 Text Notes 5700 1000 2    60   ~ 0
-X-Axis Stepper Driver
+E1 Stepper Driver
 Text GLabel 5400 9250 2    60   UnSpc ~ 0
-Z_REF
+E3_REF
 Text GLabel 10650 9250 2    60   UnSpc ~ 0
-E0_REF
+E4_REF
 Text GLabel 10650 4050 2    60   UnSpc ~ 0
-Y_REF
+E2_REF
 Text GLabel 5400 4050 2    60   UnSpc ~ 0
-X_REF
+E1_REF
 Text GLabel 12100 2500 0    60   Input ~ 0
 TWD0
@@
 TWCK0
 Text GLabel 12950 2050 0    60   UnSpc ~ 0
-Y_REF
+E2_REF
 Text GLabel 12150 2750 0    60   UnSpc ~ 0
-X_REF
+E1_REF
 Text GLabel 15300 2750 2    60   UnSpc ~ 0
-E0_REF
+E4_REF
 Text GLabel 14650 2050 2    60   UnSpc ~ 0
-Z_REF
+E3_REF
 $Comp
 L GND #PWR017
@@
 +3.3V
 Text GLabel 2250 3750 0    60   Output ~ 0
-X_EN
+E1_EN
 Text GLabel 7500 3750 0    60   Output ~ 0
-Y_EN
+E2_EN
 Text GLabel 7500 8950 0    60   Output ~ 0
-E0_EN
+E4_EN
 Text GLabel 2250 8950 0    60   Output ~ 0
-Z_EN
+E3_EN
 $Comp
 L GND #PWR018
@@
 V_IN
 Text GLabel 2250 8450 0    60   Input ~ 0
-Z_STEP
+E3_STEP
 Text GLabel 2250 8600 0    60   Input ~ 0
-Z_DIR
+E3_DIR
 Text GLabel 5250 8100 2    60   Output ~ 0
-Z_MOT_1A
+E3_MOT_1A
 Text GLabel 5250 7950 2    60   Output ~ 0
-Z_MOT_1B
+E3_MOT_1B
 Text GLabel 5250 8450 2    60   Output ~ 0
-Z_MOT_2A
+E3_MOT_2A
 Text GLabel 5250 8600 2    60   Output ~ 0
-Z_MOT_2B
+E3_MOT_2B
 Text GLabel 10500 8600 2    60   Output ~ 0
-E0_MOT_2B
+E4_MOT_2B
 Text GLabel 10500 8450 2    60   Output ~ 0
-E0_MOT_2A
+E4_MOT_2A
 Text GLabel 10500 7950 2    60   Output ~ 0
-E0_MOT_1B
+E4_MOT_1B
 Text GLabel 10500 8100 2    60   Output ~ 0
-E0_MOT_1A
+E4_MOT_1A
 Text GLabel 7500 8600 0    60   Input ~ 0
-E0_DIR
+E4_DIR
 Text GLabel 7500 8450 0    60   Input ~ 0
-E0_STEP
+E4_STEP
 Text GLabel 8650 6350 1    60   Input ~ 0
 V_IN
@@
 V_IN
 Text GLabel 7500 3250 0    60   Input ~ 0
-Y_STEP
+E2_STEP
 Text GLabel 7500 3400 0    60   Input ~ 0
-Y_DIR
+E2_DIR
 Text GLabel 10500 2900 2    60   Output ~ 0
-Y_MOT_1A
+E2_MOT_1A
 Text GLabel 10500 2750 2    60   Output ~ 0
-Y_MOT_1B
+E2_MOT_1B
 Text GLabel 10500 3250 2    60   Output ~ 0
-Y_MOT_2A
+E2_MOT_2A
 Text GLabel 10500 3400 2    60   Output ~ 0
-Y_MOT_2B
+E2_MOT_2B
 Text GLabel 5250 3400 2    60   Output ~ 0
-X_MOT_2B
+E1_MOT_2B
 Text GLabel 5250 3250 2    60   Output ~ 0
-X_MOT_2A
+E1_MOT_2A
 Text GLabel 5250 2750 2    60   Output ~ 0
-X_MOT_1B
+E1_MOT_1B
 Text GLabel 5250 2900 2    60   Output ~ 0
-X_MOT_1A
+E1_MOT_1A
 Text GLabel 2250 3400 0    60   Input ~ 0
-X_DIR
+E1_DIR
 Text GLabel 2250 3250 0    60   Input ~ 0
-X_STEP
+E1_STEP
 Text GLabel 3400 1150 1    60   Input ~ 0
 V_IN

Commit message: About 75% of the schematic changes made.
Parts:
- added SJ? (x16): MS1, symbol SJ
Connections:
- wire segments 392 -> 444

Commit message: Inputs and outputs tidied to keep DRC a bit happier...
Parts:
- gave numbers to parts that had none: 16
Connections:
- wire segments 444 -> 447
- no-connect marks 0 -> 1
Changed lines of the file:
@@
-EESchema Schematic File Version 2  date Thu 06 Nov 2014 16:31:39 GMT
+EESchema Schematic File Version 2  date Fri 07 Nov 2014 11:38:16 GMT
 LIBS:power
 LIBS:device
@@
 Sheet 2 4
 Title "Duet"
-Date "6 nov 2014"
+Date "7 nov 2014"
 Rev "0.7"
 Comp "Think3DPrint3D, RepRapPro"
@@
 Comment4 ""
 $EndDescr
+NoConn ~ 14500 2500
+Wire Wire Line
+	4950 8700 4950 8600
+Wire Wire Line
+	4950 8700 4750 8700
 Wire Wire Line
 	4950 8400 4950 8500
@@
 	4800 2700 4800 2600
 Wire Wire Line
-	4350 8600 4150 8600
+	4150 8600 4350 8600
 Wire Wire Line
 	4150 8600 4150 8500
@@
 	9400 8600 9600 8600
 Wire Wire Line
-	5250 8600 4950 8600
+	4950 8600 5250 8600
 Wire Wire Line
 	4300 7950 4350 7950
@@
 	4400 8400 4350 8400
 Connection ~ 4350 8400
-$Comp
-L SJ SJ?
+Wire Wire Line
+	4350 8600 4350 8700
+$Comp
+L SJ SJ10
 U 1 1 545B6581
 P 4550 8700
-F 0 "SJ?" H 4650 8850 50  0000 C CNN
+F 0 "SJ10" H 4650 8850 50  0000 C CNN
 F 1 "MS1" H 4650 8551 40  0000 C CNN
 	1    4550 8700
@@
 $EndComp
 $Comp
-L SJ SJ?
+L SJ SJ16
 U 1 1 545B657C
 P 4600 8400
-F 0 "SJ?" H 4700 8550 50  0000 C CNN
+F 0 "SJ16" H 4700 8550 50  0000 C CNN
 F 1 "MS1" H 4700 8251 40  0000 C CNN
 	1    4600 8400
@@
 $EndComp
 $Comp
-L SJ SJ?
+L SJ SJ15
 U 1 1 545B6579
 P 4600 8150
-F 0 "SJ?" H 4700 8300 50  0000 C CNN
+F 0 "SJ15" H 4700 8300 50  0000 C CNN
 F 1 "MS1" H 4700 8001 40  0000 C CNN
 	1    4600 8150
@@
 $EndComp
 $Comp
-L SJ SJ?
+L SJ SJ9
 U 1 1 545B6566
 P 4550 7850
-F 0 "SJ?" H 4650 8000 50  0000 C CNN
+F 0 "SJ9" H 4650 8000 50  0000 C CNN
 F 1 "MS1" H 4650 7701 40  0000 C CNN
 	1    4550 7850
@@
 $EndComp
 $Comp
-L SJ SJ?
+L SJ SJ19
 U 1 1 545B651E
 P 9800 8700
-F 0 "SJ?" H 9900 8850 50  0000 C CNN
+F 0 "SJ19" H 9900 8850 50  0000 C CNN
 F 1 "MS1" H 9900 8551 40  0000 C CNN
 	1    9800 8700
@@
 $EndComp
 $Comp
-L SJ SJ?
+L SJ SJ24
 U 1 1 545B651C
 P 9850 8400
-F 0 "SJ?" H 9950 8550 50  0000 C CNN
+F 0 "SJ24" H 9950 8550 50  0000 C CNN
 F 1 "MS1" H 9950 8251 40  0000 C CNN
 	1    9850 8400
@@
 $EndComp
 $Comp
-L SJ SJ?
+L SJ SJ23
 U 1 1 545B6517
 P 9850 8150
-F 0 "SJ?" H 9950 8300 50  0000 C CNN
+F 0 "SJ23" H 9950 8300 50  0000 C CNN
 F 1 "MS1" H 9950 8001 40  0000 C CNN
 	1    9850 8150
@@
 $EndComp
 $Comp
-L SJ SJ?
+L SJ SJ18
 U 1 1 545B6510
 P 9800 7850
-F 0 "SJ?" H 9900 8000 50  0000 C CNN
+F 0 "SJ18" H 9900 8000 50  0000 C CNN
 F 1 "MS1" H 9900 7701 40  0000 C CNN
 	1    9800 7850
@@
 $EndComp
 $Comp
-L SJ SJ?
+L SJ SJ22
 U 1 1 545B64D4
 P 9850 3500
-F 0 "SJ?" H 9950 3650 50  0000 C CNN
+F 0 "SJ22" H 9950 3650 50  0000 C CNN
 F 1 "MS1" H 9950 3351 40  0000 C CNN
 	1    9850 3500
@@
 $EndComp
 $Comp
-L SJ SJ?
+L SJ SJ21
 U 1 1 545B64D0
 P 9850 3200
-F 0 "SJ?" H 9950 3350 50  0000 C CNN
+F 0 "SJ21" H 9950 3350 50  0000 C CNN
 F 1 "MS1" H 9950 3051 40  0000 C CNN
 	1    9850 3200
@@
 $EndComp
 $Comp
-L SJ SJ?
+L SJ SJ20
 U 1 1 545B64CA
 P 9850 2950
-F 0 "SJ?" H 9950 3100 50  0000 C CNN
+F 0 "SJ20" H 9950 3100 50  0000 C CNN
 F 1 "MS1" H 9950 2801 40  0000 C CNN
 	1    9850 2950
@@
 $EndComp
 $Comp
-L SJ SJ?
+L SJ SJ17
 U 1 1 545B64BB
 P 9800 2650
-F 0 "SJ?" H 9900 2800 50  0000 C CNN
+F 0 "SJ17" H 9900 2800 50  0000 C CNN
 F 1 "MS1" H 9900 2501 40  0000 C CNN
 	1    9800 2650
@@
 $EndComp
 $Comp
-L SJ SJ?
+L SJ SJ14
 U 1 1 545B62DB
 P 4600 3500
-F 0 "SJ?" H 4700 3650 50  0000 C CNN
+F 0 "SJ14" H 4700 3650 50  0000 C CNN
 F 1 "MS1" H 4700 3351 40  0000 C CNN
 	1    4600 3500
@@
 $EndComp
 $Comp
-L SJ SJ?
+L SJ SJ13
 U 1 1 545B62D5
 P 4600 3200
-F 0 "SJ?" H 4700 3350 50  0000 C CNN
+F 0 "SJ13" H 4700 3350 50  0000 C CNN
 F 1 "MS1" H 4700 3051 40  0000 C CNN
 	1    4600 3200
@@
 $EndComp
 $Comp
-L SJ SJ?
+L SJ SJ12
 U 1 1 545B62D0
 P 4600 2950
-F 0 "SJ?" H 4700 3100 50  0000 C CNN
+F 0 "SJ12" H 4700 3100 50  0000 C CNN
 F 1 "MS1" H 4700 2801 40  0000 C CNN
 	1    4600 2950
@@
 $EndComp
 $Comp
-L SJ SJ?
+L SJ SJ11
 U 1 1 545B617B
 P 4600 2600
-F 0 "SJ?" H 4700 2750 50  0000 C CNN
+F 0 "SJ11" H 4700 2750 50  0000 C CNN
 F 1 "MS1" H 4700 2451 40  0000 C CNN
 	1    4600 2600
@@
 	1    0    0    -1
 $EndComp
-Text GLabel 13200 9150 2    39   Output ~ 0
+Text GLabel 13200 9150 2    39   Input ~ 0
 E3_STOP_CONN
 $Comp
@@
 	0    -1   -1   0
 $EndComp
-Text GLabel 15050 9150 2    39   Output ~ 0
+Text GLabel 15050 9150 2    39   Input ~ 0
 E4_STOP_CONN
-Text GLabel 13200 6550 2    39   Output ~ 0
+Text GLabel 13200 6550 2    39   Input ~ 0
 E2_STOP_CONN
 $Comp
@@
 	0    -1   -1   0
 $EndComp
-Text GLabel 15100 6550 2    39   Output ~ 0
+Text GLabel 15100 6550 2    39   Input ~ 0
 E1_STOP_CONN
 $Comp
@@
 Text Notes 5700 1000 2    60   ~ 0
 E1 Stepper Driver
-Text GLabel 5400 9250 2    60   UnSpc ~ 0
+Text GLabel 5400 9250 2    60   Input ~ 0
 E3_REF
-Text GLabel 10650 9250 2    60   UnSpc ~ 0
+Text GLabel 10650 9250 2    60   Input ~ 0
 E4_REF
-Text GLabel 10650 4050 2    60   UnSpc ~ 0
+Text GLabel 10650 4050 2    60   Input ~ 0
 E2_REF
-Text GLabel 5400 4050 2    60   UnSpc ~ 0
+Text GLabel 5400 4050 2    60   Input ~ 0
 E1_REF
 Text GLabel 12100 2500 0    60   Input ~ 0
@@
 Text GLabel 12150 2350 0    60   Input ~ 0
 TWCK0
-Text GLabel 12950 2050 0    60   UnSpc ~ 0
+Text GLabel 12950 2050 0    60   Output ~ 0
 E2_REF
-Text GLabel 12150 2750 0    60   UnSpc ~ 0
+Text GLabel 12150 2750 0    60   Output ~ 0
 E1_REF
-Text GLabel 15300 2750 2    60   UnSpc ~ 0
+Text GLabel 15300 2750 2    60   Output ~ 0
 E4_REF
-Text GLabel 14650 2050 2    60   UnSpc ~ 0
+Text GLabel 14650 2050 2    60   Output ~ 0
 E3_REF
 $Comp
@@
 Text GLabel 13750 1150 1    60   Input ~ 0
 +3.3V
-Text GLabel 2250 3750 0    60   Output ~ 0
+Text GLabel 2250 3750 0    60   Input ~ 0
 E1_EN
-Text GLabel 7500 3750 0    60   Output ~ 0
+Text GLabel 7500 3750 0    60   Input ~ 0
 E2_EN
-Text GLabel 7500 8950 0    60   Output ~ 0
+Text GLabel 7500 8950 0    60   Input ~ 0
 E4_EN
-Text GLabel 2250 8950 0    60   Output ~ 0
+Text GLabel 2250 8950 0    60   Input ~ 0
 E3_EN
 $Comp
