File: Duet-0.7/Stepper_Drv.sch (KiCad schematic (older format))
At the start: 110 parts, among them J16 VREF, J17 VREF, J18 VREF, J3 VREF, U5 A4982SLPTR, U6 A4982SLPTR, U7 A4982SLPTR, U8 A4982SLPTR, U9 MCP44X1

Commit message: New version of Duet 0.7 - Duet 0.7a with ground plane, no chokes, and stepper and heater pin headers in the same places as on the Duet 0.6.
Parts:
- removed L1, L10, L11, L12, L13, L14, L8, L9: CM_CHOKE, symbol CM_CHOKE
Connections:
- wire segments 392 -> 384
