File: Shield-0.2/Stepper_Drv.sch (KiCad schematic (older format))
At the start: 64 parts, among them J17 VREF, J3 VREF, U5 A4982SLPTR, U7 A4982SLPTR, U9 MCP44X1

Commit message: Shield: swapped the location of P1 with J2 and J4, to make it easier to connect the hotend fan looms; removed chokes
Parts:
- removed L1, L11, L12, L8: CM_CHOKE, symbol CM_CHOKE
- removed SJ11, SJ12, SJ13, SJ14, SJ17, SJ20, SJ21, SJ22: MS1, symbol SJ
Connections:
- wire segments 242 -> 217
Changed lines of the file:
@@
 	4150 3950 4150 3800
 Wire Wire Line
-	10200 3500 10200 3400
-Wire Wire Line
-	10200 3500 10050 3500
-Wire Wire Line
-	10200 3200 10200 3300
-Wire Wire Line
-	10200 3200 10050 3200
-Wire Wire Line
-	10200 2950 10200 2850
-Wire Wire Line
-	10200 2950 10050 2950
-Wire Wire Line
-	10200 2700 10200 2750
-Wire Wire Line
-	10200 2700 10000 2700
-Wire Wire Line
-	10000 2700 10000 2650
-Wire Wire Line
-	4950 3500 4950 3400
-Wire Wire Line
-	4950 3500 4800 3500
+	10200 3000 10200 2850
 Wire Wire Line
 	4950 3200 4950 3300
 Wire Wire Line
-	4950 3200 4800 3200
-Connection ~ 4350 2950
-Wire Wire Line
-	4400 2950 4350 2950
+	4350 3200 4950 3200
 Wire Wire Line
 	4950 2700 4950 2750
@@
 	4950 2700 4800 2700
 Wire Wire Line
-	4800 2700 4800 2600
-Wire Wire Line
 	5250 2900 5100 2900
 Wire Wire Line
-	10200 2750 10500 2750
+	9750 2750 10500 2750
 Wire Wire Line
 	5050 3100 5050 3050
 Wire Wire Line
-	4300 3400 4350 3400
-Wire Wire Line
 	4150 3000 4350 3000
-Wire Wire Line
-	4350 3000 4350 2850
-Wire Wire Line
-	9550 3400 9600 3400
 Wire Wire Line
 	10500 3100 10500 3050
@@
 Connection ~ 10300 3300
 Wire Wire Line
-	10200 3300 10350 3300
-Wire Wire Line
-	9400 3150 9600 3150
-Wire Wire Line
-	9600 3150 9600 3300
+	10050 3300 10350 3300
+Wire Wire Line
+	9400 3150 10050 3150
 Wire Wire Line
 	9400 3300 9550 3300
@@
 	10350 3250 10500 3250
 Wire Wire Line
-	9400 2850 9550 2850
-Wire Wire Line
-	9550 2850 9550 2750
-Wire Wire Line
-	9400 3000 9600 3000
-Wire Wire Line
-	9600 3000 9600 2850
+	9400 2850 9750 2850
+Wire Wire Line
+	9400 3000 10200 3000
 Wire Wire Line
 	10300 3050 10300 3100
@@
 Connection ~ 7100 2150
 Wire Wire Line
-	10200 3400 10500 3400
-Wire Wire Line
-	9550 2750 9600 2750
-Wire Wire Line
-	4300 2750 4350 2750
+	9550 3400 10500 3400
+Wire Wire Line
+	4300 2750 4800 2750
 Wire Wire Line
 	4150 3150 4350 3150
 Wire Wire Line
-	4350 3150 4350 3300
-Wire Wire Line
-	4950 3400 5250 3400
+	4300 3400 5250 3400
 Wire Wire Line
 	5050 3050 5250 3050
@@
 	4950 2750 5250 2750
 Wire Wire Line
-	4400 2600 4350 2600
-Wire Wire Line
-	4350 2600 4350 2750
-Wire Wire Line
 	4950 2850 4950 2950
 Wire Wire Line
-	4950 2950 4800 2950
-Wire Wire Line
-	4400 3200 4350 3200
-Connection ~ 4350 3200
-Wire Wire Line
-	4350 3400 4350 3500
-Wire Wire Line
-	4350 3500 4400 3500
-Wire Wire Line
-	9600 2750 9600 2650
-Wire Wire Line
-	9650 2950 9600 2950
-Connection ~ 9600 2950
-Wire Wire Line
-	9650 3200 9600 3200
-Connection ~ 9600 3200
-Wire Wire Line
-	9650 3500 9600 3500
-Wire Wire Line
-	9600 3500 9600 3400
+	4950 2950 4350 2950
 Wire Wire Line
 	4300 3550 4150 3550
@@
 NoConn ~ 14500 2500
 $Comp
-L SJ SJ22
-U 1 1 545B64D4
-P 9850 3500
-F 0 "SJ22" H 9950 3650 50  0000 C CNN
-F 1 "MS1" H 9950 3351 40  0000 C CNN
-F 2 "" H 9850 3500 60  0001 C CNN
-F 3 "" H 9850 3500 60  0001 C CNN
-	1    9850 3500
-	0    -1   -1   0
-$EndComp
-$Comp
-L SJ SJ21
-U 1 1 545B64D0
-P 9850 3200
-F 0 "SJ21" H 9950 3350 50  0000 C CNN
-F 1 "MS1" H 9950 3051 40  0000 C CNN
-F 2 "" H 9850 3200 60  0001 C CNN
-F 3 "" H 9850 3200 60  0001 C CNN
-	1    9850 3200
-	0    -1   -1   0
-$EndComp
-$Comp
-L SJ SJ20
-U 1 1 545B64CA
-P 9850 2950
-F 0 "SJ20" H 9950 3100 50  0000 C CNN
-F 1 "MS1" H 9950 2801 40  0000 C CNN
-F 2 "" H 9850 2950 60  0001 C CNN
-F 3 "" H 9850 2950 60  0001 C CNN
-	1    9850 2950
-	0    -1   -1   0
-$EndComp
-$Comp
-L SJ SJ17
-U 1 1 545B64BB
-P 9800 2650
-F 0 "SJ17" H 9900 2800 50  0000 C CNN
-F 1 "MS1" H 9900 2501 40  0000 C CNN
-F 2 "" H 9800 2650 60  0001 C CNN
-F 3 "" H 9800 2650 60  0001 C CNN
-	1    9800 2650
-	0    -1   -1   0
-$EndComp
-$Comp
-L SJ SJ14
-U 1 1 545B62DB
-P 4600 3500
-F 0 "SJ14" H 4700 3650 50  0000 C CNN
-F 1 "MS1" H 4700 3351 40  0000 C CNN
-F 2 "" H 4600 3500 60  0001 C CNN
-F 3 "" H 4600 3500 60  0001 C CNN
-	1    4600 3500
-	0    1    1    0
-$EndComp
-$Comp
-L SJ SJ13
-U 1 1 545B62D5
-P 4600 3200
-F 0 "SJ13" H 4700 3350 50  0000 C CNN
-F 1 "MS1" H 4700 3051 40  0000 C CNN
-F 2 "" H 4600 3200 60  0001 C CNN
-F 3 "" H 4600 3200 60  0001 C CNN
-	1    4600 3200
-	0    1    1    0
-$EndComp
-$Comp
-L SJ SJ12
-U 1 1 545B62D0
-P 4600 2950
-F 0 "SJ12" H 4700 3100 50  0000 C CNN
-F 1 "MS1" H 4700 2801 40  0000 C CNN
-F 2 "" H 4600 2950 60  0001 C CNN
-F 3 "" H 4600 2950 60  0001 C CNN
-	1    4600 2950
-	0    1    1    0
-$EndComp
-$Comp
-L SJ SJ11
-U 1 1 545B617B
-P 4600 2600
-F 0 "SJ11" H 4700 2750 50  0000 C CNN
-F 1 "MS1" H 4700 2451 40  0000 C CNN
-F 2 "" H 4600 2600 60  0001 C CNN
-F 3 "" H 4600 2600 60  0001 C CNN
-	1    4600 2600
-	0    1    1    0
-$EndComp
-$Comp
 L GND #PWR01
 U 1 1 53B05215
@@
 $EndComp
 $Comp
-L CM_CHOKE L12
-U 1 1 53B0520E
-P 9900 3400
-F 0 "L12" V 9850 3400 40  0000 C CNN
-F 1 "CM_CHOKE" V 10050 3400 40  0000 C CNN
-F 2 "" H 9900 3400 60  0001 C CNN
-F 3 "" H 9900 3400 60  0001 C CNN
-	1    9900 3400
-	0    -1   -1   0
-$EndComp
-$Comp
-L CM_CHOKE L11
-U 1 1 53B0520D
-P 9900 2850
-F 0 "L11" V 9850 2850 40  0000 C CNN
-F 1 "CM_CHOKE" V 10050 2850 40  0000 C CNN
-F 2 "" H 9900 2850 60  0001 C CNN
-F 3 "" H 9900 2850 60  0001 C CNN
-	1    9900 2850
-	0    -1   -1   0
-$EndComp
-$Comp
 L GND #PWR04
 U 1 1 53B0520A
@@
 	1    4900 2600
 	1    0    0    -1
-$EndComp
-$Comp
-L CM_CHOKE L8
-U 1 1 53B05203
-P 4650 3400
-F 0 "L8" V 4600 3400 40  0000 C CNN
-F 1 "CM_CHOKE" V 4800 3400 40  0000 C CNN
-F 2 "" H 4650 3400 60  0001 C CNN
-F 3 "" H 4650 3400 60  0001 C CNN
-	1    4650 3400
-	0    -1   -1   0
-$EndComp
-$Comp
-L CM_CHOKE L1
-U 1 1 53B05202
-P 4650 2850
-F 0 "L1" V 4600 2850 40  0000 C CNN
-F 1 "CM_CHOKE" V 4800 2850 40  0000 C CNN
-F 2 "" H 4650 2850 60  0001 C CNN
-F 3 "" H 4650 2850 60  0001 C CNN
-	1    4650 2850
-	0    -1   -1   0
 $EndComp
 $Comp
@@
 Wire Wire Line
 	12200 2350 12200 2400
+Wire Wire Line
+	4350 3150 4350 3200
+Wire Wire Line
+	4350 2950 4350 3000
+Wire Wire Line
+	4800 2750 4800 2700
+Wire Wire Line
+	9750 2850 9750 2750
+Wire Wire Line
+	10050 3150 10050 3300
 $EndSCHEMATC
