File: Duet-0.8/Headers.sch (KiCad schematic (older format))
At the start: 15 parts, among them J1 EXPANSION, J10 E0 MOT/STOP, J2 CONN2, J20 5V_PS, J23 POWER IN, J24 GND V_IN, J28 Probe, J4 BED HEATER, J5 BED TEMP, J6 CONN2, J7 Z MOT/STOP, J8 Y MOT/STOP, J9 X MOT/STOP, P1 CONN_4

Commit message: Duet Version 0.8 ----------------
Schematic changed; board still needs to be updated.

Changes:

Probe rewired to use AD12 and AD14, (standard P2 probe in the Firmware)
Bed connector - both spades and screw terminals used
Power connector - both spades and screw terminals used
Spurious power LEDS removed - there is now only one set
5V connector removed.  PS on is now a single pin.
Second Z connector added in series with the first.
Parts:
- removed J20: 5V_PS, symbol CONN_3
- removed J23: POWER IN, symbol CONN2
- removed J4: BED HEATER, symbol CONN2
- added J11: BED-, symbol SPADE1
- added J12, J4: V+, symbol SPADE1
- added J13: GND, symbol SPADE1
- added J14: BED POWER, symbol CONN2
- added J20: POWER IN, symbol CONN2
- added J23: Z MOT 2, symbol CONN_4
- added P2: CONN_1, symbol CONN_1
- C1: value CP1 -> 10u
Connections:
- net labels removed: 5V_IN, PC10
- wire segments 239 -> 251
Other:
- note added: "Bed \nConnectors"
- note added: "Power\nIn"
- note removed: "High Current\nScrew Term"
- moved on the sheet: C1, J28, J5, J7
