File: Duet-0.8/Processor.sch (KiCad schematic (older format))
At the start: 42 parts, among them J21 JTAG, J26 GND, U1 ATSAM3X8E, X2 CRYSTAL_4PIN

Commit message: This is the first complete version.  But it has not been checked for errors.
Connections:
- wire segments 161 -> 164
Changed lines of the file:
@@
 Connection ~ 14800 13850
 Wire Wire Line
-	14800 13850 14800 14000
+	14800 13850 14800 14100
 Connection ~ 14800 7000
 Wire Wire Line
-	14800 6950 14800 7000
+	14800 6800 14800 7000
 Connection ~ 14800 7550
 Wire Wire Line
@@
 Wire Wire Line
 	14850 7000 14750 7000
-Wire Wire Line
-	14750 14100 14750 14000
-Wire Wire Line
-	14750 14000 14850 14000
-Wire Wire Line
-	14850 14000 14850 14100
 Wire Wire Line
 	14750 14600 14750 14700
@@
 	0    -1   -1   0
 $EndComp
-Text GLabel 14800 6950 1    60   Input ~ 0
+Text GLabel 14800 6800 1    60   Input ~ 0
 +3.3V
 $Comp
@@
 	1    0    0    -1
 $EndComp
+Wire Wire Line
+	14750 14000 14850 14000
+Wire Wire Line
+	14850 14000 14850 14100
+Wire Wire Line
+	14750 14000 14750 14100
+Wire Wire Line
+	14850 7000 14850 6900
+Wire Wire Line
+	14850 6900 14750 6900
+Wire Wire Line
+	14750 6900 14750 7000
+Connection ~ 14800 6900
 $EndSCHEMATC
