File: Archive_Files/Duet-0.7b/Headers.sch (KiCad schematic (older format))
At the start: 20 parts, among them J1 EXPANSION, J10 E0 MOT/STOP, J11 BED-, J12 V+, J13 GND, J14 BED POWER, J2 CONN2, J20 POWER IN, J23 Z MOT 2, J24 GND V_IN, J25 PS 5V, J28 Probe, J4 V+, J5 BED TEMP, J6 CONN2, J7 Z MOT/STOP, J8 Y MOT/STOP, J9 X MOT/STOP, P1 CONN_4

Commit message: Tony's suggestion of re-instating the external 5V supply implemented. Power LEDS more widely spaced to allow easier access by printed light-pipe.
Parts:
- removed C1: 10u, ~, symbol CP1
- removed J11: BED-, symbol SPADE1
- removed J12, J4: V+, symbol SPADE1
- removed J13: GND, symbol SPADE1
- removed J14: BED POWER, symbol CONN2
- removed J20: POWER IN, symbol CONN2
- removed J23: Z MOT 2, symbol CONN_4
- removed J25: PS 5V, symbol CONN2
- added J20: 5V_PS, symbol CONN_3
- added J23: POWER IN, symbol CONN2
- added J4: BED HEATER, symbol CONN2
Connections:
- net labels added: PC10
- wire segments 254 -> 234
Other:
- note added: "High Current\nScrew Term"
- note removed: "Bed \nConnectors"
- note removed: "Power\nIn"
- moved on the sheet: J28, J5, J7
