File: Archive_Files/Duet-0.7b/Processor.sch (KiCad schematic (older format))
At the start: 42 parts, among them J21 JTAG, J26 GND, U1 ATSAM3X8E, X2 CRYSTAL_4PIN

Commit message: Tony's suggestion of re-instating the external 5V supply implemented. Power LEDS more widely spaced to allow easier access by printed light-pipe.
Connections:
- wire segments 164 -> 161
Changed lines of the file:
@@
 LIBS:valves
 LIBS:FE
-LIBS:Shield-cache
-LIBS:Duet0.8-cache
+LIBS:Duet0.7-cache
 EELAYER 27 0
 EELAYER END
@@
 Sheet 7 7
 Title "Duet"
-Date "18 mar 2015"
+Date "17 dec 2014"
 Rev "0.7"
 Comp "Think3DPrint3D, RepRapPro"
@@
 Connection ~ 14800 13850
 Wire Wire Line
-	14800 13850 14800 14100
+	14800 13850 14800 14000
 Connection ~ 14800 7000
 Wire Wire Line
-	14800 6800 14800 7000
+	14800 6950 14800 7000
 Connection ~ 14800 7550
 Wire Wire Line
@@
 Wire Wire Line
 	14850 7000 14750 7000
+Wire Wire Line
+	14750 14100 14750 14000
+Wire Wire Line
+	14750 14000 14850 14000
+Wire Wire Line
+	14850 14000 14850 14100
 Wire Wire Line
 	14750 14600 14750 14700
@@
 	0    -1   -1   0
 $EndComp
-Text GLabel 14800 6800 1    60   Input ~ 0
+Text GLabel 14800 6950 1    60   Input ~ 0
 +3.3V
 $Comp
@@
 $EndComp
 $Comp
-L GND #PWR056
+L GND #PWR058
 U 1 1 50F1BF81
 P 9200 14550
-F 0 "#PWR056" H 9200 14550 30  0001 C CNN
+F 0 "#PWR058" H 9200 14550 30  0001 C CNN
 F 1 "GND" H 9200 14480 30  0001 C CNN
 F 2 "" H 9200 14550 60  0001 C CNN
@@
 $EndComp
 $Comp
-L GND #PWR057
+L GND #PWR059
 U 1 1 50F1B3A2
 P 6500 5100
-F 0 "#PWR057" H 6500 5100 30  0001 C CNN
+F 0 "#PWR059" H 6500 5100 30  0001 C CNN
 F 1 "GND" H 6500 5030 30  0001 C CNN
 F 2 "" H 6500 5100 60  0001 C CNN
@@
 VDDPLL
 $Comp
-L GND #PWR058
+L GND #PWR060
 U 1 1 50F1AE7F
 P 12350 4000
-F 0 "#PWR058" H 12350 4000 30  0001 C CNN
+F 0 "#PWR060" H 12350 4000 30  0001 C CNN
 F 1 "GND" H 12350 3930 30  0001 C CNN
 F 2 "" H 12350 4000 60  0001 C CNN
@@
 $EndComp
 $Comp
-L GND #PWR059
+L GND #PWR061
 U 1 1 50F1AB2F
 P 13850 4500
-F 0 "#PWR059" H 13850 4500 30  0001 C CNN
+F 0 "#PWR061" H 13850 4500 30  0001 C CNN
 F 1 "GND" H 13850 4430 30  0001 C CNN
 F 2 "" H 13850 4500 60  0001 C CNN
@@
 NoConn ~ 7600 9800
 $Comp
-L GND #PWR060
+L GND #PWR062
 U 1 1 50F13953
 P 13400 14500
-F 0 "#PWR060" H 13400 14500 30  0001 C CNN
+F 0 "#PWR062" H 13400 14500 30  0001 C CNN
 F 1 "GND" H 13400 14430 30  0001 C CNN
 F 2 "" H 13400 14500 60  0001 C CNN
@@
 $EndComp
 $Comp
-L GND #PWR061
+L GND #PWR063
 U 1 1 50F1392E
 P 13400 13750
-F 0 "#PWR061" H 13400 13750 30  0001 C CNN
+F 0 "#PWR063" H 13400 13750 30  0001 C CNN
 F 1 "GND" H 13400 13680 30  0001 C CNN
 F 2 "" H 13400 13750 60  0001 C CNN
@@
 $EndComp
 $Comp
-L GND #PWR062
+L GND #PWR064
 U 1 1 505DBB16
 P 11050 15700
-F 0 "#PWR062" H 11050 15700 30  0001 C CNN
+F 0 "#PWR064" H 11050 15700 30  0001 C CNN
 F 1 "GND" H 11050 15630 30  0001 C CNN
 F 2 "" H 11050 15700 60  0001 C CNN
@@
 SPI0_SPCK
 $Comp
-L GND #PWR063
+L GND #PWR065
 U 1 1 5057A432
 P 14800 14850
-F 0 "#PWR063" H 14800 14850 30  0001 C CNN
+F 0 "#PWR065" H 14800 14850 30  0001 C CNN
 F 1 "GND" H 14800 14780 30  0001 C CNN
 F 2 "" H 14800 14850 60  0001 C CNN
@@
 $EndComp
 $Comp
-L GND #PWR064
+L GND #PWR066
 U 1 1 50579E73
 P 7550 9950
-F 0 "#PWR064" H 7550 9950 30  0001 C CNN
+F 0 "#PWR066" H 7550 9950 30  0001 C CNN
 F 1 "GND" H 7550 9880 30  0001 C CNN
 F 2 "" H 7550 9950 60  0001 C CNN
@@
 +3.3V
 $Comp
-L GND #PWR065
+L GND #PWR067
 U 1 1 5057957F
 P 8250 6600
-F 0 "#PWR065" H 8250 6600 30  0001 C CNN
+F 0 "#PWR067" H 8250 6600 30  0001 C CNN
 F 1 "GND" H 8250 6530 30  0001 C CNN
 F 2 "" H 8250 6600 60  0001 C CNN
@@
 	1    0    0    -1
 $EndComp
-Wire Wire Line
-	14750 14000 14850 14000
-Wire Wire Line
-	14850 14000 14850 14100
-Wire Wire Line
-	14750 14000 14750 14100
-Wire Wire Line
-	14850 7000 14850 6900
-Wire Wire Line
-	14850 6900 14750 6900
-Wire Wire Line
-	14750 6900 14750 7000
-Connection ~ 14800 6900
 $EndSCHEMATC
