File: Shield-0.4/Headers.sch (KiCad schematic (older format))
At the start: 22 parts, among them J1 EXPANSION, J10 E0 COOL, J11 E0 TEMP, J12 E1 H&T, J13 FAN_0, J14 E0 MOT/STOP, J15 E0 MOT/STOP, J16 CONN2, J19 E0 HEAT, J2 PWR, J24 PWR, J28 Probe, J4 PWR, J5 E2 H&T, J6 SPADE1, J7 SPADE1, J8 E2 MOT/STOP, J9 E1 MOT/STOP, P1 STEP, P2 E0 H&T

Commit message: Shield V0.4 - WIP
Parts:
- removed J16: CONN2, symbol CONN2
- removed J2, J24: PWR, symbol CONN2
Changed lines of the file:
@@
 Sheet 3 4
 Title "Duet"
-Date "17 dec 2014"
+Date "6 mar 2015"
 Rev "0.7"
 Comp "Think3DPrint3D, RepRapPro"
@@
 +3.3V
 $Comp
-L GND #PWR22
+L GND #PWR018
 U 1 1 545B8A07
 P 7400 3150
-F 0 "#PWR22" H 7400 3150 30  0001 C CNN
+F 0 "#PWR018" H 7400 3150 30  0001 C CNN
 F 1 "GND" H 7400 3080 30  0001 C CNN
 F 2 "" H 7400 3150 60  0001 C CNN
@@
 VSSA
 $Comp
-L GND #PWR19
+L GND #PWR019
 U 1 1 545B85D0
 P 1600 10750
-F 0 "#PWR19" H 1600 10750 30  0001 C CNN
+F 0 "#PWR019" H 1600 10750 30  0001 C CNN
 F 1 "GND" H 1600 10680 30  0001 C CNN
 F 2 "" H 1600 10750 60  0001 C CNN
@@
 	1    2150 10500
 	1    0    0    1
-$EndComp
-$Comp
-L CONN2 J2
-U 1 1 545B85C7
-P 2150 10100
-F 0 "J2" H 2150 10000 40  0000 C CNN
-F 1 "PWR" V 2300 10150 40  0000 C CNN
-F 2 "" H 2150 10100 60  0001 C CNN
-F 3 "" H 2150 10100 60  0001 C CNN
-	1    2150 10100
-	1    0    0    1
-$EndComp
-Text GLabel 1600 10100 0    60   Input ~ 0
-V_IN
-$Comp
-L GND #PWR18
-U 1 1 545B85C6
-P 1600 10350
-F 0 "#PWR18" H 1600 10350 30  0001 C CNN
-F 1 "GND" H 1600 10280 30  0001 C CNN
-F 2 "" H 1600 10350 60  0001 C CNN
-F 3 "" H 1600 10350 60  0001 C CNN
-	1    1600 10350
-	1    0    0    -1
 $EndComp
 $Comp
@@
 $EndComp
 $Comp
-L GND #PWR23
+L GND #PWR021
 U 1 1 545B7245
 P 12050 5950
-F 0 "#PWR23" H 12050 5950 30  0001 C CNN
+F 0 "#PWR021" H 12050 5950 30  0001 C CNN
 F 1 "GND" H 12050 5880 30  0001 C CNN
 F 2 "" H 12050 5950 60  0001 C CNN
@@
 PROBE-SIG
 $Comp
-L GND #PWR17
-U 1 1 53B0339C
-P 1600 9900
-F 0 "#PWR17" H 1600 9900 30  0001 C CNN
-F 1 "GND" H 1600 9830 30  0001 C CNN
-F 2 "" H 1600 9900 60  0001 C CNN
-F 3 "" H 1600 9900 60  0001 C CNN
-	1    1600 9900
-	1    0    0    -1
-$EndComp
-$Comp
-L GND #PWR21
+L GND #PWR023
 U 1 1 53B0339B
 P 4300 5800
-F 0 "#PWR21" H 4300 5800 30  0001 C CNN
+F 0 "#PWR023" H 4300 5800 30  0001 C CNN
 F 1 "GND" H 4300 5730 30  0001 C CNN
 F 2 "" H 4300 5800 60  0001 C CNN
@@
 	1    0    0    -1
 $EndComp
-Text GLabel 1600 9650 0    60   Input ~ 0
-V_IN
-$Comp
-L CONN2 J24
-U 1 1 53B03332
-P 2150 9650
-F 0 "J24" H 2150 9550 40  0000 C CNN
-F 1 "PWR" V 2300 9700 40  0000 C CNN
-F 2 "" H 2150 9650 60  0001 C CNN
-F 3 "" H 2150 9650 60  0001 C CNN
-	1    2150 9650
-	1    0    0    1
-$EndComp
-$Comp
-L GND #PWR20
+$Comp
+L GND #PWR024
 U 1 1 5220B9D2
 P 4100 9900
-F 0 "#PWR20" H 4100 9900 30  0001 C CNN
+F 0 "#PWR024" H 4100 9900 30  0001 C CNN
 F 1 "GND" H 4100 9830 30  0001 C CNN
 F 2 "" H 4100 9900 60  0001 C CNN
@@
 V_IN
 $Comp
-L GND #PWR16
+L GND #PWR025
 U 1 1 5064C39B
 P 1100 950
-F 0 "#PWR16" H 1100 950 30  0001 C CNN
+F 0 "#PWR025" H 1100 950 30  0001 C CNN
 F 1 "GND" H 1100 880 30  0001 C CNN
 F 2 "" H 1100 950 60  0001 C CNN
@@
 	4450 5950 4650 5950
 Wire Wire Line
-	1800 9750 1600 9750
-Wire Wire Line
-	1600 9750 1600 9900
-Wire Wire Line
 	1600 7150 1850 7150
 Wire Wire Line
@@
 	1850 1900 1600 1900
 Wire Wire Line
-	1600 9650 1800 9650
-Wire Wire Line
 	4400 5650 4650 5650
 Wire Wire Line
@@
 	6150 2600 5450 2600
 Wire Wire Line
-	1600 10100 1800 10100
-Wire Wire Line
-	1600 10350 1600 10200
-Wire Wire Line
-	1600 10200 1800 10200
-Wire Wire Line
 	1800 10600 1600 10600
 Wire Wire Line
@@
 	13900 3200 14100 3200
 Wire Wire Line
-	14100 3150 14100 3350
-Wire Wire Line
 	14050 1800 12800 1800
 Wire Wire Line
@@
 Wire Wire Line
 	13950 1700 13750 1700
-$Comp
-L CONN2 J16
-U 1 1 5491609A
-P 14450 3450
-F 0 "J16" H 14450 3350 40  0000 C CNN
-F 1 "CONN2" V 14600 3500 40  0000 C CNN
-F 2 "" H 14450 3450 60  0000 C CNN
-F 3 "" H 14450 3450 60  0000 C CNN
-	1    14450 3450
-	1    0    0    -1
-$EndComp
 Connection ~ 14100 3200
-Wire Wire Line
-	14100 3450 14000 3450
-Wire Wire Line
-	14000 3450 14000 3000
 Connection ~ 14000 3000
 $Comp
@@
 Wire Wire Line
 	3050 5700 3100 5700
+Wire Wire Line
+	14100 3200 14100 3150
 $EndSCHEMATC

Commit message: Yet more WIP...
Parts:
- added J18: E3 MOT/STOP, symbol CONN7
- added J20: E4 MOT/STOP, symbol CONN7
Connections:
- net +3.3V: now also J18.6 (P6), J20.6 (P6)
- net GND: now also J18.7 (P7), J20.7 (P7)
- new net E3_MOT_1A: J18.2 (P2)
- new net E3_MOT_1B: J18.1 (P1)
- new net E3_MOT_2A: J18.3 (P3)
- new net E3_MOT_2B: J18.4 (P4)
- new net E3_STOP_CONN: J18.5 (P5)
- new net E4_MOT_1A: J20.2 (P2)
- new net E4_MOT_1B: J20.1 (P1)
- new net E4_MOT_2A: J20.3 (P3)
- new net E4_MOT_2B: J20.4 (P4)
- new net E4_STOP_CONN: J20.5 (P5)
Changed lines of the file:
@@
 Sheet 3 4
 Title "Duet"
-Date "6 mar 2015"
+Date "10 mar 2015"
 Rev "0.7"
 Comp "Think3DPrint3D, RepRapPro"
@@
 +3.3V
 $Comp
-L GND #PWR018
+L GND #PWR37
 U 1 1 545B8A07
 P 7400 3150
-F 0 "#PWR018" H 7400 3150 30  0001 C CNN
+F 0 "#PWR37" H 7400 3150 30  0001 C CNN
 F 1 "GND" H 7400 3080 30  0001 C CNN
 F 2 "" H 7400 3150 60  0001 C CNN
@@
 VSSA
 $Comp
-L GND #PWR019
+L GND #PWR33
 U 1 1 545B85D0
 P 1600 10750
-F 0 "#PWR019" H 1600 10750 30  0001 C CNN
+F 0 "#PWR33" H 1600 10750 30  0001 C CNN
 F 1 "GND" H 1600 10680 30  0001 C CNN
 F 2 "" H 1600 10750 60  0001 C CNN
@@
 $EndComp
 $Comp
-L GND #PWR021
+L GND #PWR38
 U 1 1 545B7245
 P 12050 5950
-F 0 "#PWR021" H 12050 5950 30  0001 C CNN
+F 0 "#PWR38" H 12050 5950 30  0001 C CNN
 F 1 "GND" H 12050 5880 30  0001 C CNN
 F 2 "" H 12050 5950 60  0001 C CNN
@@
 PROBE-SIG
 $Comp
-L GND #PWR023
+L GND #PWR35
 U 1 1 53B0339B
 P 4300 5800
-F 0 "#PWR023" H 4300 5800 30  0001 C CNN
+F 0 "#PWR35" H 4300 5800 30  0001 C CNN
 F 1 "GND" H 4300 5730 30  0001 C CNN
 F 2 "" H 4300 5800 60  0001 C CNN
@@
 $EndComp
 $Comp
-L GND #PWR024
+L GND #PWR34
 U 1 1 5220B9D2
 P 4100 9900
-F 0 "#PWR024" H 4100 9900 30  0001 C CNN
+F 0 "#PWR34" H 4100 9900 30  0001 C CNN
 F 1 "GND" H 4100 9830 30  0001 C CNN
 F 2 "" H 4100 9900 60  0001 C CNN
@@
 V_IN
 $Comp
-L GND #PWR025
+L GND #PWR32
 U 1 1 5064C39B
 P 1100 950
-F 0 "#PWR025" H 1100 950 30  0001 C CNN
+F 0 "#PWR32" H 1100 950 30  0001 C CNN
 F 1 "GND" H 1100 880 30  0001 C CNN
 F 2 "" H 1100 950 60  0001 C CNN
@@
 Wire Wire Line
 	14100 3200 14100 3150
+Text GLabel 7450 3750 1    60   Input ~ 0
++3.3V
+$Comp
+L GND #PWR36
+U 1 1 54FF6056
+P 7350 5950
+F 0 "#PWR36" H 7350 5950 30  0001 C CNN
+F 1 "GND" H 7350 5880 30  0001 C CNN
+F 2 "" H 7350 5950 60  0001 C CNN
+F 3 "" H 7350 5950 60  0001 C CNN
+	1    7350 5950
+	1    0    0    -1
+$EndComp
+$Comp
+L CONN7 J18
+U 1 1 54FF605C
+P 9750 4200
+F 0 "J18" H 9750 3900 50  0000 C CNN
+F 1 "E3 MOT/STOP" V 9800 4200 40  0000 C CNN
+F 2 "" H 9750 4200 60  0001 C CNN
+F 3 "" H 9750 4200 60  0001 C CNN
+	1    9750 4200
+	1    0    0    -1
+$EndComp
+$Comp
+L CONN7 J20
+U 1 1 54FF6062
+P 9750 5150
+F 0 "J20" H 9750 4850 50  0000 C CNN
+F 1 "E4 MOT/STOP" V 9800 5150 40  0000 C CNN
+F 2 "" H 9750 5150 60  0001 C CNN
+F 3 "" H 9750 5150 60  0001 C CNN
+	1    9750 5150
+	1    0    0    -1
+$EndComp
+Text GLabel 8250 5400 0    60   Output ~ 0
+E4_STOP_CONN
+Text GLabel 8250 4450 0    60   Output ~ 0
+E3_STOP_CONN
+Text GLabel 8250 4950 0    60   Input ~ 0
+E4_MOT_1A
+Text GLabel 8250 4800 0    60   Input ~ 0
+E4_MOT_1B
+Text GLabel 8250 5100 0    60   Input ~ 0
+E4_MOT_2A
+Text GLabel 8250 5250 0    60   Input ~ 0
+E4_MOT_2B
+Text GLabel 8250 4300 0    60   Input ~ 0
+E3_MOT_2B
+Text GLabel 8250 4150 0    60   Input ~ 0
+E3_MOT_2A
+Text GLabel 8250 3850 0    60   Input ~ 0
+E3_MOT_1B
+Text GLabel 8250 4000 0    60   Input ~ 0
+E3_MOT_1A
+Wire Wire Line
+	7350 5950 7350 4700
+Wire Wire Line
+	9400 4400 9300 4400
+Wire Wire Line
+	9300 4400 9300 4600
+Wire Wire Line
+	9300 4600 7450 4600
+Wire Wire Line
+	9400 4200 9200 4200
+Wire Wire Line
+	9200 4200 9200 4300
+Wire Wire Line
+	9200 4300 8250 4300
+Wire Wire Line
+	9400 4000 8250 4000
+Wire Wire Line
+	9400 3900 8550 3900
+Wire Wire Line
+	9400 5350 9300 5350
+Wire Wire Line
+	9300 5350 9300 5550
+Wire Wire Line
+	9300 5550 7450 5550
+Wire Wire Line
+	9400 5150 9200 5150
+Wire Wire Line
+	9200 5150 9200 5250
+Wire Wire Line
+	9200 5250 8250 5250
+Wire Wire Line
+	9400 4950 8250 4950
+Connection ~ 7450 4600
+Connection ~ 7350 5700
+Wire Wire Line
+	7350 5700 9350 5700
+Wire Wire Line
+	8250 5400 9250 5400
+Wire Wire Line
+	8250 5100 9150 5100
+Wire Wire Line
+	8250 4800 8500 4800
+Wire Wire Line
+	8250 4450 9250 4450
+Wire Wire Line
+	8250 4150 9150 4150
+Wire Wire Line
+	8250 3850 8500 3850
+Wire Wire Line
+	8500 4800 8550 4850
+Wire Wire Line
+	8500 3850 8550 3900
+Wire Wire Line
+	7350 4700 9350 4700
+Connection ~ 7450 5550
+Connection ~ 7350 4700
+Wire Wire Line
+	8550 4850 9400 4850
+Wire Wire Line
+	9150 5100 9150 5050
+Wire Wire Line
+	9150 5050 9400 5050
+Wire Wire Line
+	9250 5400 9250 5250
+Wire Wire Line
+	9250 5250 9400 5250
+Wire Wire Line
+	9350 5700 9350 5450
+Wire Wire Line
+	9350 5450 9400 5450
+Wire Wire Line
+	9150 4150 9150 4100
+Wire Wire Line
+	9150 4100 9400 4100
+Wire Wire Line
+	9250 4450 9250 4300
+Wire Wire Line
+	9250 4300 9400 4300
+Wire Wire Line
+	9350 4700 9350 4500
+Wire Wire Line
+	9350 4500 9400 4500
+Wire Wire Line
+	7450 5550 7450 3750
 $EndSCHEMATC

Commit message: Shield V0.4.  First complete design.
Parts:
- added J21: PWR, symbol CONN2
Connections:
- net GND: now also J21.1 (P1)
- net V_IN: now also J21.2 (PM)
Changed lines of the file:
@@
 Sheet 3 4
 Title "Duet"
-Date "18 mar 2015"
+Date "25 mar 2015"
 Rev "0.7"
 Comp "Think3DPrint3D, RepRapPro"
@@
 Wire Wire Line
 	7450 5550 7450 3750
+$Comp
+L GND #PWR041
+U 1 1 5512F625
+P 1600 9900
+F 0 "#PWR041" H 1600 9900 30  0001 C CNN
+F 1 "GND" H 1600 9830 30  0001 C CNN
+F 2 "" H 1600 9900 60  0001 C CNN
+F 3 "" H 1600 9900 60  0001 C CNN
+	1    1600 9900
+	1    0    0    -1
+$EndComp
+Text GLabel 1600 9650 0    60   Input ~ 0
+V_IN
+$Comp
+L CONN2 J21
+U 1 1 5512F62C
+P 2150 9650
+F 0 "J21" H 2150 9550 40  0000 C CNN
+F 1 "PWR" V 2300 9700 40  0000 C CNN
+F 2 "" H 2150 9650 60  0001 C CNN
+F 3 "" H 2150 9650 60  0001 C CNN
+	1    2150 9650
+	1    0    0    1
+$EndComp
+Wire Wire Line
+	1800 9750 1600 9750
+Wire Wire Line
+	1600 9750 1600 9900
+Wire Wire Line
+	1600 9650 1800 9650
 $EndSCHEMATC
