File: Shield-0.4/Stepper_Drv.sch (KiCad schematic (older format))
At the start: 52 parts, among them J17 VREF, J3 VREF, U5 A4982SLPTR, U7 A4982SLPTR, U9 MCP44X1

Commit message: Shield V0.4 - WIP
Parts:
- removed SJ1, SJ3: MS2, symbol SJ
- removed SJ2, SJ4: MS1, symbol SJ
Connections:
- wire segments 217 -> 219

Commit message: Yet more WIP...
Parts:
- added C13, C21, C33, C39: 0u22, symbol C
- added C15, C17, C23, C31, C35, C38, C42, C47: 0u1, symbol C
- added C16, C37: 100u, symbol C_POL
- added C25, C27, C28, C29, C43, C44, C45, C46: 47n, symbol C_SMALL
- added J16, J2: VREF, symbol VREF
- added R10, R11, R15, R16: 0R1, symbol R
- added R12: 100k, 0603, symbol R
- added R13, R8: 10k, symbol R
- added R14, R9: 0R, symbol R
- added R7: 100k, symbol R
- added U1, U2: A4982SLPTR, symbol A4982SLPTR
Connections:
- net +3.3V: now also C21.1, C39.1, R12.1, R13.1, R7.1, R8.1, U1.10 (VDD), U1.5 (MS1), U1.6 (MS2), U2.10 (VDD), U2.5 (MS1), U2.6 (MS2)
- net E3_REF: now also C31.1, J2.1 (Vref), U1.12 (REF)
- net E4_REF: now also C47.1, J16.1 (Vref), U2.12 (REF)
- net GND: now also C13.2, C15.1, C16.2, C21.2, C25.1, C27.2, C28.1, C29.2, C31.2, C33.2, C35.1, C37.2, C39.2, C43.1, C44.2, C45.1, C46.2, C47.2, R10.2, R11.2, R14.2, R15.2, R16.2, R9.2, U1.13 (GND), U1.24 (GND), U1.25 (GND_PAD), U1.26 (GND), U1.27 (GND), U1.28 (GND), U1.29 (GND), U1.30 (GND), U1.31 (GND), U1.32 (GND), U1.33 (GND), U1.34 (GND), U2.13 (GND), U2.24 (GND), U2.25 (GND_PAD), U2.26 (GND), U2.27 (GND), U2.28 (GND), U2.29 (GND), U2.30 (GND), U2.31 (GND), U2.32 (GND), U2.33 (GND), U2.34 (GND)
- net V_IN: now also C15.2, C16.1, C17.2, C35.2, C37.1, C38.2, U1.16 (VBB1), U1.21 (VBB2), U2.16 (VBB1), U2.21 (VBB2)
- new net: C42.1, U2.1 (CP1)
- new net: C42.2, U2.2 (CP2)
- new net: C23.1, U1.1 (CP1)
- new net: C23.2, U1.2 (CP2)
- new net: R16.1, U2.17 (SENSE1)
- new net: R15.1, U2.20 (SENSE2)
- new net: C38.1, U2.3 (VCP)
- new net: C33.1, U2.4 (VREG)
- new net: R13.2, U2.7 (/RESET), U2.9 (/SLEEP)
- new net: R14.1, U2.8 (ROSC)
- new net: R11.1, U1.17 (SENSE1)
- new net: R10.1, U1.20 (SENSE2)
- new net: C17.1, U1.3 (VCP)
- new net: C13.1, U1.4 (VREG)
- new net: R8.2, U1.7 (/RESET), U1.9 (/SLEEP)
- new net: R9.1, U1.8 (ROSC)
- new net E3_DIR: U1.14 (DIR)
- new net E3_EN: R7.2, U1.23 (/ENABLE)
- new net E3_MOT_1A: C27.1, U1.18 (OUT1A)
- new net E3_MOT_1B: C25.2, U1.15 (OUT1B)
- new net E3_MOT_2A: C28.2, U1.19 (OUT2A)
- new net E3_MOT_2B: C29.1, U1.22 (OUT2B)
- new net E3_STEP: U1.11 (STEP)
- new net E4_DIR: U2.14 (DIR)
- new net E4_EN: R12.2, U2.23 (/ENABLE)
- new net E4_MOT_1A: C44.1, U2.18 (OUT1A)
- new net E4_MOT_1B: C43.2, U2.15 (OUT1B)
- new net E4_MOT_2A: C45.2, U2.19 (OUT2A)
- new net E4_MOT_2B: C46.1, U2.22 (OUT2B)
- new net E4_STEP: U2.11 (STEP)

Commit message: Shield WIP.
Parts:
- added C48, C49: 0u1, symbol C_SMALL
- added D5, D8: LED, symbol LED
- added R17, R25: 100R, symbol R_SMALL
- added R24, R28: 680R, symbol R
Connections:
- net +3.3V: now also R24.2, R28.2
- net GND: now also C48.2, C49.2
- new net: D8.1 (A), R28.1
- new net: D5.1 (A), R24.1
- new net E3_STOP: C48.1, R17.1
- new net E3_STOP_CONN: D5.2 (K), R17.2
- new net E4_STOP: C49.1, R25.1
- new net E4_STOP_CONN: D8.2 (K), R25.2
