File: Duet_Expansion/Expansion_Breakoutv1.1/ExpBreakout.sch (KiCad schematic (older format))
At the start: 18 parts, among them J1 EXPANSION, P1 E2, P2 E3, P3 E4, P4 E5, P5 E6, P6 H6_PWM, P7 H7_PWM, U1 75ALS192, U2 75ALS192, U3 75ALS192, U4 75ALS192, U5 74HCT02

Commit message: Rename to v1.1
Expansion Breakout board version was incorrect at v1.0 (that was a in house development version) Verison 1.1 is the shipped version.
Parts:
- P1, P2, P3, P4, P5: symbol CONN_01X06 -> Conn_01x06
- P6, P7: symbol CONN_01X03 -> Conn_01x03
Changed lines of the file:
@@
 encoding utf-8
 Sheet 1 1
-Title "Duet Wifi"
+Title "Expansion Breakout"
 Date "02 Jul 2016"
-Rev "1.0"
+Rev "1.1"
 Comp "Think3DPrint3D, Escher 3D"
 Comment1 "CERN OSH License 1.2"
@@
 NoConn ~ 6490 8080
 $Comp
-L CONN_01X06 P1
+L Conn_01x06 P1
 U 1 1 5899A6E8
 P 9300 2000
@@
 	9000 1950 9100 1950
 $Comp
-L CONN_01X06 P2
+L Conn_01x06 P2
 U 1 1 5899C06D
 P 9300 3050
@@
 	9000 3000 9100 3000
 $Comp
-L CONN_01X06 P3
+L Conn_01x06 P3
 U 1 1 5899C0E8
 P 9300 4150
@@
 	9000 4100 9100 4100
 $Comp
-L CONN_01X06 P4
+L Conn_01x06 P4
 U 1 1 5899C163
 P 9300 5200
@@
 	9000 5150 9100 5150
 $Comp
-L CONN_01X06 P5
+L Conn_01x06 P5
 U 1 1 5899C3DB
 P 9300 6250
@@
 $EndComp
 $Comp
-L CONN_01X03 P7
+L Conn_01x03 P7
 U 1 1 58C9053E
 P 9270 9220
@@
 $EndComp
 $Comp
-L CONN_01X03 P6
+L Conn_01x03 P6
 U 1 1 58C90747
 P 9260 8460
